Commit message: Add in tennis ball launcher

File: entertrainer_test/urdf/dog.urdf (robot description, URDF)
Before this commit: robot dog, 2 links, 1 joints
Links:
- link body: geometry collision box size=0.5 1 0.25; visual box size=0.5 1 0.25
- link front_left_leg: geometry collision sphere radius=0.0625; visual sphere radius=0.0625
Joints:
- removed joint front_joint
- added joint base_to_right_leg: type continuous, parent body, child front_left_leg, origin xyz=-0.125 -0.4375 -0.1875, axis 0 1 0

File: entertrainer_test/urdf/tennis_ball.urdf (robot description, URDF)
Before this commit: robot tennis_ball, 1 links, 0 joints
Links:
- removed link ball
- added link ball_body, mass 0.0585; collision sphere radius=0.01905; visual sphere radius=0.01905
