Commit message: Making the test twist not crash into table

File: entertrainer_test/urdf/tennis_ball.urdf (robot description, URDF)
Before this commit: robot tennis_ball, 1 links, 0 joints
Links:
- link ball: geometry collision sphere radius=0.0343; visual sphere radius=0.0343

Commit message: adding robot model

File: entertrainer_test/urdf/tennis_ball.urdf (robot description, URDF)
Before this commit: robot tennis_ball, 1 links, 0 joints
Links:
- link ball_body: mass 0.0585 -> 0.0498
