Commit message: Adding in some stencils

File: entertrainer_test/urdf/vase.urdf (robot description, URDF)
Before this commit: robot dog, 1 links, 0 joints
Links:
- link base_link: geometry collision box size=0.266 0.266 0.5; visual mesh filename=package://entertrainer_test/urdf/stl/lava_vase1.stl scale=0.125 0.125 0.125

Commit message: Deconflicting the navigation and exploration files

File: entertrainer_test/urdf/vase.urdf (robot description, URDF)
Before this commit: robot vase, 1 links, 0 joints
Links:
- link base_link: geometry collision box size=0.266 0.266 0.35; visual mesh filename=package://entertrainer_test/urdf/stl/lava_vase1.stl scale=0.06125 0.06125 0.06125
