Commit message: Working through integration, collision detection launcher distance, and rviz look better

File: entertrainer_test/urdf/robot/turtlebot3_waffle.urdf.xacro (robot description, xacro)
@@ -199,5 +199,5 @@
   <link name="camera_rgb_frame"/>
   <joint name="camera_rgb_optical_joint" type="fixed">
-    <origin xyz="0 0 0" rpy="-1.57 0 -1.57"/>
+    <origin xyz="0 0 0" rpy="0 0 0"/>
     <parent link="camera_rgb_frame"/>
     <child link="camera_rgb_optical_frame"/>
