Commit message: Setting up the Entertrainer Base for usage

File: entertrainer_test/urdf/robot/entertrainer.gazebo.xacro (robot description, xacro)
@@ -105,5 +105,5 @@
     <material>Gazebo/FlatBlack</material>
     <sensor type="ray" name="lds_lfcd_sensor">
-      <pose>0 0 0 0 0 0</pose>
+      <pose>0 0 0 0 0 0</pose><!--0 0 0 0 0 0-->
       <visualize>$(arg laser_visual)</visualize>
       <update_rate>5</update_rate>

File: entertrainer_test/urdf/robot/turtlebot3_waffle.urdf.xacro (robot description, xacro)
@@ -1,6 +1,6 @@
 <?xml version="1.0" ?>
-<robot name="entertrainer" xmlns:xacro="http://ros.org/wiki/xacro">
-  <xacro:include filename="$(find entertrainer_test)/urdf/robot/common_properties.xacro"/>
-  <xacro:include filename="$(find entertrainer_test)/urdf/robot/entertrainer.gazebo.xacro"/>
+<robot name="turtlebot3_waffle" xmlns:xacro="http://ros.org/wiki/xacro">
+  <xacro:include filename="$(find turtlebot3_description)/urdf/common_properties.xacro"/>
+  <xacro:include filename="$(find turtlebot3_description)/urdf/turtlebot3_waffle.gazebo.xacro"/>
   <xacro:property name="r200_cam_rgb_px" value="0.005"/>
   <xacro:property name="r200_cam_rgb_py" value="0.018"/>
@@ -11,22 +11,19 @@
     <parent link="base_footprint"/>
     <child link="base_link" />
-    <origin xyz="0 0 0" rpy="0 0 1.57"/>
+    <origin xyz="0 0 0.010" rpy="0 0 0"/>
   </joint>
   <link name="base_link">
     <visual>
-      <origin xyz="0 0 0.14" rpy="0 0 0"/>
-<!--      <origin xyz="-0.064 0 0.16" rpy="0 0 1.57"/>
--->
-      <geometry>
-        <mesh filename="package://entertrainer_test/urdf/stl/Entertrainertrybodycombined.stl" scale="0.025 0.025 0.025"/>
-        <!-- <mesh filename="package://turtlebot3_description/meshes/bases/waffle_base.stl" scale="0.001 0.001 0.001"/> -->
+      <origin xyz="-0.09 0 0.14" rpy="0 0 1.57"/>
+<!--      <origin xyz="-0.064 0 0.0" rpy="0 0 0"/>-->
+      <geometry>
+        <mesh filename="package://entertrainer_test/urdf/stl/Entertrainertrybodycombined.stl" scale="0.0295 0.0235 0.0235"/>
       </geometry>
       <material name="light_black"/>
     </visual>
     <collision>
-      <!--<origin xyz="-0.064 0 0.047" rpy="0 0 0"/>-->
-      <origin xyz="0 0 0.1" rpy="0 0 0"/>
-      <geometry>
-        <box size="0.206 0.266 0.094"/>
+      <origin xyz="-0.064 0 0.047" rpy="0 0 0"/>
+      <geometry>
+        <box size="0.266 0.266 0.094"/>
       </geometry>
     </collision>
@@ -42,15 +39,12 @@
     <parent link="base_link"/>
     <child link="wheel_left_link"/>
-    <origin xyz="0.115 -0.090 0.025" rpy="0 1.57 0"/>
+    <origin xyz="0.0 0.144 0.023" rpy="-1.57 0 0"/>
     <axis xyz="0 0 1"/>
   </joint>
   <link name="wheel_left_link">
     <visual>
-    <!--  <origin xyz="-0.25 0.0 -0.3" rpy="1.57 1.57 0"/>
-    <origin xyz="0 0 -0.0625" rpy="0 3.14 0"/>-->
-<!--    <origin xyz="-0.1095 -0.090 0.025" rpy="0 -1.57 3.14"/>-->
-      <origin xyz="0.09 -0.116 -0.10" rpy="1.57 1.57 0"/>
-      <geometry>
-        <mesh filename="package://entertrainer_test/urdf/stl/weels.stl" scale="0.025 0.025 0.025"/>
+      <origin xyz="0 0 0" rpy="1.57 0 0"/>
+      <geometry>
+        <mesh filename="package://turtlebot3_description/meshes/wheels/left_tire.stl" scale="0.001 0.001 0.001"/>
       </geometry>
       <material name="dark"/>
@@ -59,5 +53,5 @@
       <origin xyz="0 0 0" rpy="0 0 0"/>
       <geometry>
-        <cylinder length="0.018" radius="0.04"/>
+        <cylinder length="0.018" radius="0.033"/>
       </geometry>
     </collision>
@@ -73,14 +67,12 @@
     <parent link="base_link"/>
     <child link="wheel_right_link"/>
-    <origin xyz="-0.115 -0.090 0.025" rpy="0 1.57 3.14"/>
+    <origin xyz="0.0 -0.144 0.023" rpy="-1.57 0 0"/>
     <axis xyz="0 0 1"/>
   </joint>
   <link name="wheel_right_link">
     <visual>
-      <origin xyz="0.09 -0.116 -0.10" rpy="1.57 1.57 0"/>
-<!--      <origin xyz="0.14 0.125 0.11" rpy="1.57 0 1.57"/>
--->
-      <geometry>
-        <mesh filename="package://entertrainer_test/urdf/stl/weels.stl" scale="0.025 0.025 0.025"/>
+      <origin xyz="0 0 0" rpy="1.57 0 0"/>
+      <geometry>
+        <mesh filename="package://turtlebot3_description/meshes/wheels/right_tire.stl" scale="0.001 0.001 0.001"/>
       </geometry>
       <material name="dark"/>
@@ -89,5 +81,5 @@
       <origin xyz="0 0 0" rpy="0 0 0"/>
       <geometry>
-        <cylinder length="0.018" radius="0.04"/>
+        <cylinder length="0.018" radius="0.033"/>
       </geometry>
     </collision>
@@ -103,6 +95,5 @@
     <parent link="base_link"/>
     <child link="caster_back_right_link"/>
-    <origin xyz="0 0.068 -0.004" rpy="-1.57 0 -1.57"/>
-    <!-- <origin xyz="0 0.068 -0.004" rpy="-1.57 0 0"/>-->
+    <origin xyz="-0.177 -0.064 -0.004" rpy="-1.57 0 0"/>
   </joint>
   <link name="caster_back_right_link">
@@ -121,5 +112,5 @@
     </inertial>
   </link>
-<!--  <joint name="caster_back_left_joint" type="fixed">
+  <joint name="caster_back_left_joint" type="fixed">
     <parent link="base_link"/>
     <child link="caster_back_left_link"/>
@@ -140,5 +131,5 @@
                izz="0.001" />
     </inertial>
-  </link>-->
+  </link>
   <joint name="imu_joint" type="fixed">
     <parent link="base_link"/>
@@ -152,5 +143,5 @@
     <origin xyz="-0.064 0 0.122" rpy="0 0 0"/>
   </joint>
-  <link name="base_scan">
+  <link name="base_scan"><!-- 360 Lidar-->
     <visual>
       <origin xyz="0 0 0" rpy="0 0 0"/>

Commit message: fixing point cloud rviz

File: entertrainer_test/urdf/robot/entertrainer.gazebo.xacro (robot description, xacro)
@@ -156,5 +156,6 @@
         <updateRate>30.0</updateRate>
         <cameraName>camera</cameraName>
-        <frameName>camera_rgb_optical_frame</frameName>
+        <frameName>depth_tf_frame</frameName>
+        <!--<frameName>camera_rgb_optical_frame</frameName>-->
         <imageTopicName>rgb/image_raw</imageTopicName>
         <depthImageTopicName>depth/image_raw</depthImageTopicName>

File: entertrainer_test/urdf/robot/turtlebot3_waffle.urdf.xacro (robot description, xacro)
@@ -8,4 +8,15 @@
   <xacro:property name="r200_cam_depth_offset" value="0.01"/>
   <link name="base_footprint"/>
+  <joint name="depth_tf" type="fixed">
+    <!--red  X axis,
+          green is Y,
+            blue is Z-->
+    <origin xyz="0 0 0.1" rpy="-1.57 0 -1.57"/>
+<!--    <origin xyz="0 2 0.1" rpy="-1.57 1.57 -1.57"/>
+-->
+    <parent link="base_footprint"/>
+    <child link="depth_tf_frame"/>
+  </joint>
+  <link name="depth_tf_frame"/>
   <joint name="base_joint" type="fixed">
     <parent link="base_footprint"/>
